File: Flash Mother Board/Flash Mother Board.kicad_pcb (KiCad board)
At the start: 2 copper layers, 1.6 x 9.8 mm, 32 parts, among them IC1 RP2040_QFN56, IC2 AZ1117CH-3.3TRG1, J1 104031-0811, SW1 KMR2, SW2 KMR2, U1 W25Q128JV, U2 W25Q128JV, X1 microUSB, Y1 12MHZ

Commit message: Last one I swear
Parts:
- moved SW2 19.2 mm to (43.0, 104.0)
- moved IC2 2.83 mm to (53.0, 96.0)
- moved D1 1.00 mm to (23.0, 85.0)
Changed lines of the file:
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@@
   )
   (footprint "Adafruit ItsyBitsy RP2040:SOD-323F" (layer "F.Cu")
-    (at 23 86)
+    (at 23 85)
     (property "Sheetfile" "Flash Mother Board.kicad_sch")
     (property "Sheetname" "")
@@
   )
   (footprint "3.3VRegForUSB:SOT230P700X180-4N" (layer "F.Cu")
-    (at 51 98)
+    (at 53 96)
     (descr "SOT-223-")
     (tags "Integrated Circuit")
@@
   )
   (footprint "Adafruit ItsyBitsy RP2040:BTN_KMR2_4.6X2.8" (layer "F.Cu")
-    (at 60.3 95.57 90)
-    (property "Sheetfile" "Flash Mother Board.kicad_sch")
-    (property "Sheetname" "")
+    (at 43 104 90)
+    (property "Sheetfile" "Flash Mother Board.kicad_sch")
+    (property "Sheetname" "")

Commit message: Routing Almost Complete
Parts:
- moved U2 119.4 mm to (206.5, 70.2)
- moved U1 53.7 mm to (86.8, 61.3)
- moved R6 53.6 mm to (73.2, 69.0), turned to 180 degrees
- moved R3 53.5 mm to (88.0, 79.3)
- moved C12 53.5 mm to (81.5, 77.1)
- moved C13 53.5 mm to (81.5, 79.8)
- moved IC1 53.5 mm to (86.8, 72.4)
- moved Y1 53.5 mm to (85.4, 79.2)
- moved SW1 52.9 mm to (73.2, 75.2)
- moved J1 52.2 mm to (106.5, 64.8)
- moved D1 51.9 mm to (73.1, 71.5)
- moved TP1 47.2 mm to (63.5, 77.0)
- moved X1 41.6 mm to (59.2, 63.4)
- moved IC2 39.0 mm to (73.5, 62.8)
- moved SW2 37.7 mm to (73.2, 81.5), turned to 180 degrees
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Connections:
- R1 pad 1: Net-(R1-Pad1) -> Net-(X1-D+)
- R2 pad 1: Net-(R2-Pad1) -> Net-(X1-D-)
- R5 pad 1: SPI0_SCK -> SPI0_CS0
- X1 pad 1: (no net) -> VBUS
- X1 pad 2: (no net) -> Net-(X1-D+)
- X1 pad 3: (no net) -> Net-(X1-D-)
- X1 pad 4: (no net) -> unconnected-(X1-ID-Pad4)
- X1 pad 5: (no net) -> GND
Routing:
- net SPI0_MOSI: track 70.0 -> 174.0 mm, vias 2 -> 4
- net SPI0_SCK: track 68.6 -> 169.9 mm, vias 2 -> 4
- net SPI0_MISO: track 70.5 -> 168.9 mm, vias 2 -> 4
- net SPI0_CS0: track 66.7 -> 163.3 mm, vias 2 -> 4
- net GND: track 8.49 -> 51.2 mm, vias 8 -> 19
- net +3V3: track 3.77 -> 46.0 mm, vias 2 -> 18
- net /D-: track 0.00 -> 28.7 mm, vias 0 -> 2
- net SPI0_CS1: track 91.4 -> 64.0 mm
- net /D+: track 0.00 -> 25.8 mm, vias 0 -> 2
- net /~{RESET}: track 0.00 -> 25.8 mm, vias 0 -> 2
- net 1.2V: track 0.00 -> 21.9 mm, vias 0 -> 2
- net /USBBOOT: track 0.00 -> 17.1 mm
- net /QSPI_CS: track 16.0 -> 25.7 mm
- net VBUS: track 0.00 -> 7.77 mm
- net Net-(D1-PadA): track 0.00 -> 5.41 mm
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- added copper zone on In2.Cu, net +3V3
- added copper zone on B.Cu, net GND
Other:
- board size 1.6 x 9.8 mm -> 163 x 33.5 mm
- copper layers 2 -> 4
- board text added: "USB"
- board text removed: "USB_Boot"
