File: Flash Mother Board/Flash Mother Board.kicad_pcb (KiCad board)
At the start: 4 copper layers, 163 x 33.5 mm, 32 parts, among them IC1 RP2040_QFN56, IC2 AZ1117CH-3.3TRG1, J1 104031-0811, SW1 KMR2, SW2 KMR2, U1 W25Q128JV, U2 W25Q128JV, X1 microUSB, Y1 12MHZ

Commit message: Banananna
Parts:
- added J2: Power Supply banannanan, Connector:Banana_Jack_2Pin, F.Cu at (121.0, 70.2)
- moved C11 1.25 mm to (66.8, 70.3)
- moved C4 1.25 mm to (66.8, 74.3)
- moved C5 1.25 mm to (62.2, 74.2)
- moved C6 1.25 mm to (66.8, 72.3)
- moved C7 1.25 mm to (62.2, 70.5)
- moved C8 1.25 mm to (62.2, 71.8)
- moved C9 1.25 mm to (62.2, 73.0)
Connections:
- U2 pad 8: +3V3 -> Net-(J2-Pin_2)
Routing:
- net Net-(J2-Pin_2): track 0.00 -> 96.4 mm, vias 0 -> 2
- net SPI0_MISO: track 168.9 -> 150.1 mm
- net SPI0_CS0: track 163.3 -> 145.8 mm, vias 4 -> 3
- net +3V3: track 46.1 -> 53.0 mm
- net GND: track 51.2 -> 52.9 mm
- net SPI0_SCK: track 169.9 -> 168.4 mm, vias 4 -> 2
- net /D+: track 25.8 -> 27.1 mm
- net (no net): track 1.19 -> 0.00 mm
- net 1.2V: track 21.9 -> 23.1 mm, vias 2 -> 0
- net /D-: track 28.7 -> 27.6 mm
- net SPI0_MOSI: track 174.0 -> 173.5 mm, vias 4 -> 2
Other:
- board size 163 x 33.5 mm -> 160.5 x 33.5 mm
