File: Flash Mother Board/Flash Mother Board.kicad_sch (KiCad schematic)
At the start: 32 parts, among them IC1 RP2040_QFN56, IC2 AZ1117CH-3.3TRG1, J1 104031-0811, SW1 KMR2, SW2 KMR2, U1 W25Q128JV, U2 W25Q128JV, X1 microUSB, Y1 12MHZ

Commit message: Banananna
Parts:
- added J2: Power Supply, Connector:Banana_Jack_2Pin, symbol Connector_Generic:Conn_01x02
Connections:
- net +3V3: no longer U2.8 (VCC)
- net GND: now also J2.1 (Pin_1)
- new net: J2.2 (Pin_2), U2.8 (VCC)
Changed lines of the file:
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@@
 	)
 	(junction
+		(at 269.24 154.94)
+		(diameter 0)
+		(color 0 0 0 0)
+	)
+	(junction
 		(at 127 30.48)
 		(diameter 0)
@@
 	(wire
 		(pts
+			(xy 269.24 142.24) (xy 269.24 147.32)
+		)
+		(stroke
+			(width 0)
+			(type default)
+		)
+	)
+	(wire
+		(pts
 			(xy 119.38 157.48) (xy 129.54 157.48)
 		)
@@
 	(wire
 		(pts
+			(xy 269.24 149.86) (xy 269.24 154.94)
+		)
+		(stroke
+			(width 0)
+			(type default)
+		)
+	)
+	(wire
+		(pts
 			(xy 273.05 44.45) (xy 275.59 44.45)
 		)
@@
 	(wire
 		(pts
-			(xy 265.43 154.94) (xy 266.7 154.94)
+			(xy 265.43 154.94) (xy 269.24 154.94)
+		)
+		(stroke
+			(width 0)
+			(type default)
+		)
+	)
+	(wire
+		(pts
+			(xy 265.43 142.24) (xy 269.24 142.24)
 		)
 		(stroke
@@
 	(wire
 		(pts
-			(xy 265.43 130.81) (xy 265.43 142.24)
+			(xy 228.6 127) (xy 228.6 128.27)
 		)
 		(stroke
@@
 	(wire
 		(pts
-			(xy 228.6 127) (xy 228.6 128.27)
+			(xy 74.803 35.56) (xy 88.138 35.56)
 		)
 		(stroke
@@
 	(wire
 		(pts
-			(xy 74.803 35.56) (xy 88.138 35.56)
+			(xy 269.24 154.94) (xy 269.24 156.21)
 		)
 		(stroke
@@
 	)
 	(symbol
-		(lib_id "Adafruit ItsyBitsy RP2040-eagle-import:GND")
-		(at 266.7 157.48 0)
-		(mirror y)
-		(unit 1)
-		(exclude_from_sim no)
-		(in_bom yes)
-		(on_board yes)
-		(dnp no)
-		(property "Reference" "#GND08"
-			(at 266.7 157.48 0)
-			(effects
-				(font
-					(size 1.27 1.27)
-				)
-				(hide yes)
-			)
-		)
-		(property "Value" "GND"
-			(at 269.24 160.02 0)
-			(effects
-				(font
-					(size 1.778 1.5113)
-				)
-				(justify left bottom)
-			)
-		)
-		(property "Footprint" "Adafruit ItsyBitsy RP2040:"
-			(at 266.7 157.48 0)
-			(effects
-				(font
-					(size 1.27 1.27)
-				)
-				(hide yes)
-			)
-		)
-		(property "Datasheet" ""
-			(at 266.7 157.48 0)
-			(effects
-				(font
-					(size 1.27 1.27)
-				)
-				(hide yes)
-			)
-		)
-		(property "Description" ""
-			(at 266.7 157.48 0)
-			(effects
-				(font
-					(size 1.27 1.27)
-				)
-				(hide yes)
-			)
-		)
-		(pin "1"
-		)
-		(instances
-			(project "Flash Mother Board"
-				(path "/f8edefc2-0888-457d-9803-46e1c7e584b2"
-					(reference "#GND08")
-					(unit 1)
-				)
-			)
-		)
-	)
-	(symbol
 		(lib_id "Adafruit ItsyBitsy RP2040-eagle-import:+3V3")
 		(at 233.68 25.908 0)
@@
 	)
 	(symbol
+		(lib_id "Connector_Generic:Conn_01x02")
+		(at 274.32 149.86 0)
+		(mirror x)
+		(unit 1)
+		(exclude_from_sim no)
+		(in_bom yes)
+		(on_board yes)
+		(dnp no)
+		(fields_autoplaced yes)
+		(property "Reference" "J2"
+			(at 274.32 140.97 0)
+			(effects
+				(font
+					(size 1.27 1.27)
+				)
+			)
+		)
+		(property "Value" "Power Supply"
+			(at 274.32 143.51 0)
+			(effects
+				(font
+					(size 1.27 1.27)
+				)
+			)
+		)
+		(property "Footprint" "Connector:Banana_Jack_2Pin"
+			(at 274.32 149.86 0)
+			(effects
+				(font
+					(size 1.27 1.27)
+				)
+				(hide yes)
+			)
+		)
+		(property "Datasheet" "~"
+			(at 274.32 149.86 0)
+			(effects
+				(font
+					(size 1.27 1.27)
+				)
+				(hide yes)
+			)
+		)
+		(property "Description" ""
+			(at 274.32 149.86 0)
+			(effects
+				(font
+					(size 1.27 1.27)
+				)
+				(hide yes)
+			)
+		)
+		(pin "1"
+		)
+		(pin "2"
+		)
+		(instances
+			(project "Flash Mother Board"
+				(path "/f8edefc2-0888-457d-9803-46e1c7e584b2"
+					(reference "J2")
+					(unit 1)
+				)
+			)
+		)
+	)
+	(symbol
 		(lib_id "Adafruit ItsyBitsy RP2040-eagle-import:RP2040_QFN56")
 		(at 81.28 147.32 0)
@@
 	)
 	(symbol
-		(lib_id "Adafruit ItsyBitsy RP2040-eagle-import:+3V3")
-		(at 265.43 128.27 0)
+		(lib_id "Adafruit ItsyBitsy RP2040-eagle-import:SPIFLASH_8PIN_4X4")
+		(at 250.19 149.86 0)
 		(unit 1)
 		(exclude_from_sim no)
@@
 		(on_board yes)
 		(dnp no)
-		(property "Reference" "#+3V09"
-			(at 265.43 128.27 0)
+		(property "Reference" "U2"
+			(at 237.49 137.16 0)
 			(effects
 				(font
-					(size 1.27 1.27)
+					(size 1.778 1.5113)
 				)
-				(hide yes)
+				(justify left bottom)
 			)
 		)
-		(property "Value" "+3V3"
-			(at 262.89 133.35 90)
+		(property "Value" "W25Q128JV"
+			(at 237.49 160.02 0)
 			(effects
 				(font
@@
 			)
 		)
-		(property "Footprint" "Adafruit ItsyBitsy RP2040:"
-			(at 265.43 128.27 0)
+		(property "Footprint" "Package_SO:SOIC-8_5.275x5.275mm_P1.27mm"
+			(at 250.19 149.86 0)
 			(effects
 				(font
@@
 		)
 		(property "Datasheet" ""
-			(at 265.43 128.27 0)
+			(at 250.19 149.86 0)
 			(effects
 				(font
@@
 		)
 		(property "Description" ""
-			(at 265.43 128.27 0)
+			(at 250.19 149.86 0)
 			(effects
 				(font
@@
 		(pin "1"
 		)
+		(pin "2"
+		)
+		(pin "3"
+		)
+		(pin "4"
+		)
+		(pin "5"
+		)
+		(pin "6"
+		)
+		(pin "7"
+		)
+		(pin "8"
+		)
+		(pin "PAD"
+		)
 		(instances
 			(project "Flash Mother Board"
 				(path "/f8edefc2-0888-457d-9803-46e1c7e584b2"
-					(reference "#+3V09")
+					(reference "U2")
 					(unit 1)
 				)
@@
 	)
 	(symbol
-		(lib_id "Adafruit ItsyBitsy RP2040-eagle-import:SPIFLASH_8PIN_4X4")
-		(at 250.19 149.86 0)
+		(lib_id "power:GND")
+		(at 40.64 190.5 0)
 		(unit 1)
 		(exclude_from_sim no)
@@
 		(on_board yes)
 		(dnp no)
-		(property "Reference" "U2"
-			(at 237.49 137.16 0)
+		(fields_autoplaced yes)
+		(property "Reference" "#PWR04"
+			(at 40.64 196.85 0)
 			(effects
 				(font
-					(size 1.778 1.5113)
+					(size 1.27 1.27)
 				)
-				(justify left bottom)
+				(hide yes)
 			)
 		)
-		(property "Value" "W25Q128JV"
-			(at 237.49 160.02 0)
+		(property "Value" "GND"
+			(at 40.64 194.6331 0)
 			(effects
 				(font
-					(size 1.778 1.5113)
+					(size 1.27 1.27)
 				)
-				(justify left bottom)
 			)
 		)
-		(property "Footprint" "Package_SO:SOIC-8_5.275x5.275mm_P1.27mm"
-			(at 250.19 149.86 0)
+		(property "Footprint" ""
+			(at 40.64 190.5 0)
 			(effects
 				(font
@@
 		)
 		(property "Datasheet" ""
-			(at 250.19 149.86 0)
+			(at 40.64 190.5 0)
 			(effects
 				(font
@@
 		)
 		(property "Description" ""
-			(at 250.19 149.86 0)
+			(at 40.64 190.5 0)
 			(effects
 				(font
@@
 		(pin "1"
 		)
-		(pin "2"
-		)
-		(pin "3"
-		)
-		(pin "4"
-		)
-		(pin "5"
-		)
-		(pin "6"
-		)
-		(pin "7"
-		)
-		(pin "8"
-		)
-		(pin "PAD"
-		)
 		(instances
 			(project "Flash Mother Board"
 				(path "/f8edefc2-0888-457d-9803-46e1c7e584b2"
-					(reference "U2")
+					(reference "#PWR04")
 					(unit 1)
 				)
@@
 	)
 	(symbol
-		(lib_id "power:GND")
-		(at 40.64 190.5 0)
+		(lib_id "Adafruit ItsyBitsy RP2040-eagle-import:GND")
+		(at 269.24 158.75 0)
 		(unit 1)
 		(exclude_from_sim no)
@@
 		(on_board yes)
 		(dnp no)
-		(fields_autoplaced yes)
-		(property "Reference" "#PWR04"
-			(at 40.64 196.85 0)
+		(property "Reference" "#GND08"
+			(at 269.24 158.75 0)
 			(effects
 				(font
@@
 		)
 		(property "Value" "GND"
-			(at 40.64 194.6331 0)
+			(at 266.7 161.29 0)
 			(effects
 				(font
-					(size 1.27 1.27)
+					(size 1.778 1.5113)
 				)
+				(justify left bottom)
 			)
 		)
-		(property "Footprint" ""
-			(at 40.64 190.5 0)
+		(property "Footprint" "Adafruit ItsyBitsy RP2040:"
+			(at 269.24 158.75 0)
 			(effects
 				(font
@@
 		)
 		(property "Datasheet" ""
-			(at 40.64 190.5 0)
+			(at 269.24 158.75 0)
 			(effects
 				(font
@@
 		)
 		(property "Description" ""
-			(at 40.64 190.5 0)
+			(at 269.24 158.75 0)
 			(effects
 				(font
@@
 			(project "Flash Mother Board"
 				(path "/f8edefc2-0888-457d-9803-46e1c7e584b2"
-					(reference "#PWR04")
+					(reference "#GND08")
 					(unit 1)
 				)
