File: Flash_Motherboard_Rev_2/Flash_Motherboard_Rev_2.kicad_pcb (KiCad board)
At the start: 4 copper layers, 9.8 x 1.6 mm, 33 parts, among them IC1 RP2040_QFN56, IC2 AZ1117CH-3.3TRG1, J1 104031-0811, J2 Power Supply, SW1 KMR2, SW2 KMR2, U1 W25Q128JV, U2 W25Q128JV, X1 microUSB, Y1 12MHZ

Commit message: Rev 2 almost done
Parts:
- added C14: 0.1uF, Capacitor_SMD:C_0402_1005Metric, F.Cu at (124.9, 100.5)
- C6: value 1uF -> 0.1uF; footprint Capacitor_SMD:C_0603_1608Metric -> Capacitor_SMD:C_0402_1005Metric
- moved U2 92.1 mm to (230.0, 94.0)
- moved X1 68.6 mm to (92.8, 89.1), turned to -90 degrees
- moved SW1 56.9 mm to (97.0, 97.6)
- moved SW2 51.1 mm to (104.0, 97.6)
- moved C10 50.1 mm to (103.0, 92.9)
- moved IC2 49.8 mm to (105.8, 88.2)
- moved D1 47.4 mm to (114.0, 94.0)
- moved C11 46.4 mm to (108.6, 92.9), turned to 180 degrees
- moved J1 35.5 mm to (144.0, 86.5), turned to 180 degrees
- moved C6 34.5 mm to (118.0, 95.4), turned to 180 degrees
- moved Y1 34.4 mm to (121.6, 100.5)
- moved U1 33.2 mm to (117.2, 86.3)
- moved TP1 32.9 mm to (109.0, 97.6)
- moved IC1 30.1 mm to (124.0, 94.3)
- moved C9 29.5 mm to (125.0, 88.0), turned to 90 degrees
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Routing:
- net /D-: track 0.00 -> 37.2 mm, vias 0 -> 2
- net /D+: track 0.00 -> 36.2 mm, vias 0 -> 2
- net /~{RESET}: track 0.00 -> 34.7 mm, vias 0 -> 2
- net +3V3: track 0.00 -> 26.5 mm, vias 0 -> 2
- net /USBBOOT: track 0.00 -> 23.9 mm
- net 1.2V: track 0.00 -> 22.5 mm, vias 0 -> 2
- net GND: track 0.00 -> 21.4 mm, vias 0 -> 23
- net /QSPI_CS: track 0.00 -> 19.1 mm
- net /QSPI_SD1: track 0.00 -> 16.3 mm
- net /QSPI_SD2: track 0.00 -> 14.8 mm
- net VBUS: track 0.00 -> 8.37 mm
- net Net-(IC1-XIN): track 0.00 -> 7.22 mm
- net /QSPI_SD3: track 0.00 -> 6.70 mm
- net Net-(C13-Pad2): track 0.00 -> 6.06 mm
- net /QSPI_SCLK: track 0.00 -> 5.28 mm
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- added copper zone on F.Cu, net +3V3
- added copper zone on B.Cu, net GND
Other:
- board size 9.8 x 1.6 mm -> 150 x 50 mm
- copper layers 4 -> 2
- board text added: "BOOT"
- board text added: "RST"

Commit message: Routing Done
Parts:
- moved U2 14.0 mm to (244.0, 92.8)
- moved TP1 5.00 mm to (114.0, 97.6)
- moved R7 3.04 mm to (134.0, 101.0)
- moved R5 2.65 mm to (132.5, 101.0)
- moved J1 0.82 mm to (144.0, 87.4)
- moved C6 0.77 mm to (118.8, 95.4)
- moved C7 0.77 mm to (118.8, 91.8)
Routing:
- net SPI0_MOSI: track 0.00 -> 147.6 mm, vias 0 -> 4
- net SPI0_SCK: track 0.00 -> 147.2 mm, vias 0 -> 2
- net SPI0_MISO: track 0.00 -> 144.9 mm, vias 0 -> 2
- net Net-(J2-Pin_2): track 0.00 -> 142.3 mm
- net SPI0_CS0: track 0.00 -> 138.9 mm, vias 0 -> 2
- net SPI0_CS1: track 1.20 -> 41.5 mm, vias 1 -> 2
- net GND: track 21.4 -> 26.6 mm
- net +3V3: track 26.5 -> 29.5 mm
Other:
- board size 150 x 50 mm -> 160 x 50 mm

Commit message: ready for review
Parts:
- moved C10 46.2 mm to (82.3, 51.6)
- moved C11 46.2 mm to (87.8, 51.6)
- moved J1 46.2 mm to (123.2, 46.1)
- moved R5 46.2 mm to (111.8, 59.8)
- moved R7 46.2 mm to (113.2, 59.8)
- moved C14 46.2 mm to (104.1, 59.2)
- moved C3 46.2 mm to (105.2, 59.2)
- moved C5 46.2 mm to (108.5, 50.5)
- moved C6 46.2 mm to (98.0, 54.1)
- moved C7 46.2 mm to (98.0, 50.5)
- moved D1 46.2 mm to (93.2, 52.8)
- moved IC2 46.2 mm to (85.0, 47.0)
- moved R4 46.2 mm to (93.8, 50.2)
- moved R6 46.2 mm to (92.8, 50.2)
- moved R8 46.2 mm to (106.2, 59.2)
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Routing:
- net Net-(J2-Pin_2): track 142.3 -> 132.9 mm
Other:
- board size 160 x 50 mm -> 160.6 x 160.6 mm
