File: RP2040_SEE/RP2040_SEE.kicad_pcb (KiCad board)
At the start: 2 copper layers, 87 x 58 mm, 4 parts, among them J1 Conn_01x20, J2 Conn_01x20, U1 Pico, U2 Pico

Commit message: banana phone
Parts:
- added J3: USB_A, Connector_USB:USB_A_TE_292303-7_Horizontal, F.Cu at (186.2, 58.9)
- added J4: USB_B_Micro, Connector_USB:USB_Micro-B_Amphenol_10103594-0001LF_Horizontal, F.Cu at (203.0, 53.9)
- added J5: Conn_01x03_Pin, Connector_PinHeader_2.54mm:PinHeader_1x03_P2.54mm_Vertical, F.Cu at (190.5, 73.0)
- added J6: Conn_01x02_Pin, Connector_PinHeader_2.54mm:PinHeader_1x02_P2.54mm_Vertical, F.Cu at (190.5, 95.0)
- moved U1 58.2 mm to (107.1, 79.9)
- moved J1 58.2 mm to (172.0, 55.7)
- moved J2 58.2 mm to (136.0, 55.7)
- moved U2 58.2 mm to (154.0, 79.9)
Connections:
- net Net-(J1-Pin_2) renamed /VSYS
Routing:
- net /VSYS: track 9.13 -> 60.9 mm
- net /D+: track 0.00 -> 25.5 mm
- net /D-: track 0.00 -> 23.5 mm
- net Net-(J4-VBUS): track 0.00 -> 21.0 mm
- net GND: track 54.7 -> 72.8 mm
- net Net-(J3-VBUS): track 0.00 -> 9.10 mm
Other:
- board size 87 x 58 mm -> 120 x 58 mm
- board text added: "GND"
- board text added: "NC"
- board text added: "USB_A V+"
- board text added: "USB_M V+"
- board text added: "VSYS"
