File: RP2040_SEE/RP2040_SEE.kicad_sch (KiCad schematic)
At the start: 4 parts, among them J1 Conn_01x20, J2 Conn_01x20, U1 Pico, U2 Pico

Commit message: banana phone
Parts:
- added J3: USB_A, Connector_USB:USB_A_TE_292303-7_Horizontal, symbol Connector:USB_A
- added J4: USB_B_Micro, Connector_USB:USB_Micro-B_Amphenol_10103594-0001LF_Horizontal, symbol Connector:USB_B_Micro
- added J5: Conn_01x03_Pin, Connector_PinHeader_2.54mm:PinHeader_1x03_P2.54mm_Vertical, symbol Connector:Conn_01x03_Pin
- added J6: Conn_01x02_Pin, Connector_PinHeader_2.54mm:PinHeader_1x02_P2.54mm_Vertical, symbol Connector:Conn_01x02_Pin
Connections:
- net GND: now also J3.4 (GND), J3.5 (Shield), J4.5 (GND), J4.6 (Shield), J6.2 (Pin_2)
- net VSYS: now reaches J1.2 (Pin_2), U2.39 (VSYS)
- net VSYS: now also J6.1 (Pin_1)
- new net: J3.1 (VBUS), J5.2 (Pin_2)
- new net: J4.1 (VBUS), J5.3 (Pin_3)
- new net D+: J3.3 (D+), J4.3 (D+)
- new net D-: J3.2 (D-), J4.2 (D-)
- no-connect marks 0 -> 1
